File: Seite01_RFID-Edelsteindetektor/schematics/Goethe_RFID_v2.sch (EAGLE design)
At the start: 61 parts, among them IC1 LM1086-ADJ, IC2 LM2937, M1 ARDUINO_R3_SMALL, Q1 IRF8313P, Q2 IRF8313P, Q3 IRF8313P, X1 12V supply

Commit message: Fix missing wire on signal LED4
Other:
- note added: "Drop D1 to allow shield to be supplied from the Unos Vin."
- note added: "TODO: Replace linear regulator with a buck regulator to decrease power dissipation."
Changed lines of the file:
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@@
 Red: 4.5R=20/4 || 47, 1/4W
 Green/Blue: 1R=2R/2,1/8W</text>
+<text x="251.46" y="332.74" size="1.778" layer="90">Drop D1 to allow shield to be
+supplied from the Unos Vin.</text>
+<text x="-25.4" y="266.7" size="1.778" layer="90">TODO:
+Replace linear regulator with a buck
+regulator to decrease power dissipation.</text>
 </plain>
 <instances>
